File: board-design/pico-ducky.kicad_pcb (KiCad board)
At the start: 2 copper layers, 36.9 x 68 mm, 9 parts, among them J1 Conn_01x20_Female, J2 Conn_01x20_Female, SW3 SK-14D01-G_6

Commit message: Added microSD reader and changed switches
Parts:
- removed SW3: SK-14D01-G_6, SK-14D01-G6:SK-14D01-G 6
- added CON1: ~, PCM_4ms_Connector_Card:CardSlot_MicroSD_YamaichiPJS008U-3000, F.Cu at (121.9, 117.8)
- added SW1: ~, PCM_CB_Devices:Slide_Switch_SPDT_P3mm_10x5x10mm, F.Cu at (106.7, 68.1)
- added SW2: ~, PCM_CB_Devices:Slide_Switch_SPDT_P3mm_10x5x10mm, F.Cu at (106.7, 80.8)
Connections:
- J1 pad 10: unconnected-(J1-Pad10) -> Net-(J1-Pin_10)
- J1 pad 11: unconnected-(J1-Pad11) -> Net-(J1-Pin_11)
- J1 pad 12: unconnected-(J1-Pad12) -> Net-(J1-Pin_12)
- J1 pad 13: Net-(J1-Pad13) -> unconnected-(J1-Pin_13-Pad13)
- J1 pad 14: Net-(J1-Pad14) -> unconnected-(J1-Pin_14-Pad14)
- J1 pad 15: Net-(J1-Pad15) -> unconnected-(J1-Pin_15-Pad15)
- J1 pad 6: Net-(J1-Pad6) -> unconnected-(J1-Pin_6-Pad6)
- J1 pad 7: Net-(J1-Pad7) -> unconnected-(J1-Pin_7-Pad7)
- J1 pad 9: unconnected-(J1-Pad9) -> Net-(J1-Pin_9)
- J2 pad 17: unconnected-(J2-Pad17) -> Net-(CON1-DAT2)
- J2 pad 18: unconnected-(J2-Pad18) -> Net-(CON1-CMD)
- J2 pad 19: unconnected-(J2-Pad19) -> Net-(CON1-CD/DAT3)
- J2 pad 5: unconnected-(J2-Pad5) -> Net-(CON1-VDD)
Routing:
- net Net-(CON1-VDD): track 0.00 -> 57.3 mm
- net Net-(CON1-CMD): track 0.00 -> 43.2 mm
- net Net-(CON1-CLK): track 0.00 -> 28.5 mm
- net Net-(CON1-DAT2): track 0.00 -> 27.4 mm
- net Net-(CON1-DAT0): track 0.00 -> 25.1 mm
- net Net-(CON1-CD/DAT3): track 0.00 -> 21.2 mm
- net Net-(J1-Pin_8): track 9.54 -> 21.4 mm
- net Net-(J1-Pad15): track 10.4 -> 0.00 mm
- net Net-(J1-Pad14): track 10.2 -> 0.00 mm
- net Net-(J1-Pad6): track 9.99 -> 0.00 mm
- net Net-(J1-Pad13): track 9.99 -> 0.00 mm
- net Net-(J1-Pad7): track 9.77 -> 0.00 mm
- net Net-(J1-Pin_12): track 0.00 -> 8.62 mm
- net Net-(J1-Pin_11): track 0.00 -> 8.43 mm
- net Net-(J1-Pin_9): track 0.00 -> 7.27 mm
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Other:
- board size 36.9 x 68 mm -> 36.9 x 78.2 mm
